File: kicad/ultim8x64.kicad_pcb (KiCad board)
At the start: 2 copper layers, 487.7 x 61 mm, 560 parts, among them P1 Input1, P10 GND, P11 5V, P12 GND, P2 Output1, P3 Input2, P4 Output2, P5 5V, P6 GND, P7 5V, P8 GND, P9 5V, U1 APA102, U10 APA102, U100 APA102, U101 APA102, U102 APA102, U103 APA102, U104 APA102, U105 APA102, U106 APA102, U107 APA102, U108 APA102, U109 APA102, U11 APA102, U110 APA102, U111 APA102, U112 APA102, U113 APA102, U114 APA102, U115 APA102, U116 APA102, U117 APA102, U118 APA102, U119 APA102, U12 APA102, U120 APA102, U121 APA102, U122 APA102, U123 APA102, U124 APA102, U125 APA102, U126 APA102, U127 APA102, U128 APA102, U129 APA102, U13 APA102, U130 APA102, U131 APA102, U132 APA102, U133 APA102, U134 APA102, U135 APA102, U136 APA102, U137 APA102, U138 APA102, U139 APA102, U14 APA102, U140 APA102, U141 APA102, U142 APA102, U143 APA102, U144 APA102, U145 APA102, U146 APA102, U147 APA102, U148 APA102, U149 APA102, U15 APA102, U150 APA102, U151 APA102, U152 APA102, U153 APA102, U154 APA102, U155 APA102, U156 APA102, U157 APA102, U158 APA102, U159 APA102, U16 APA102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

Commit message: APA102C 8x64 Panel
Routing:
- net /Row_A/5V: track 4270.9 -> 4579.4 mm, vias 120 -> 135
